File: led.d.kicad_pcb (KiCad board)
At the start: 2 copper layers, 25.4 x 30.5 mm, 5 parts, among them J1 USB_B_Micro, J2 Conn_02x02_Top_Bottom

Commit message: update
Parts:
- removed the REF** at (17.8, 38.1)
- removed RV1: Varistor_US, Varistor:RV_Disc_D7mm_W3.4mm_P5mm
- added R1000: R_US, Resistor_THT:R_Axial_DIN0204_L3.6mm_D1.6mm_P5.08mm_Horizontal, F.Cu at (77.5, 259.1)
- added REF**: OSHW-Logo2_7.3x6mm_SilkScreen, Symbol:OSHW-Logo2_7.3x6mm_SilkScreen, F.Cu at (66.1, 280.5)
- D1: moved to F.Cu
- J2: footprint Conn_02x02_Top_Bottom:Conn_02x02_Top_Bottom -> Connector_PinHeader_1.00mm:PinHeader_2x02_P1.00mm_Vertical; moved to F.Cu
- moved D1 247.6 mm to (64.2, 260.5)
- moved J1 247.6 mm to (76.8, 280.8)
- moved J2 246.3 mm to (77.5, 271.8)
Connections:
- J1 pad 6: unconnected-(J1-Pad6) -> Shiled
- J2 pad 1: data negative -> Shiled
- J2 pad 2: data positive -> data negative
- J2 pad 3: unconnected-(J2-Pad3) -> ID
- J2 pad 4: ID -> data positive
Routing:
- net Shiled: track 0.00 -> 22.6 mm
- net VCC: track 10.3 -> 32.9 mm
- net Net-(D1-Pad2): track 28.3 -> 6.28 mm
- net data positive: track 4.65 -> 5.51 mm
- net data negative: track 4.51 -> 5.36 mm
Other:
- board size 25.4 x 30.5 mm -> 26.7 x 29.7 mm
- board text added: "D+"
- board text added: "D-"
- board text added: "ID"
- board text added: "Shield"
